Commit message: adding navigation jazz

File: mpdr/urdf/mpdr.xacro (robot description, xacro)
@@ -9,5 +9,5 @@
         <visual>
             <geometry>
-                <box size="0.7112 0.7112 0.3175"/>
+                <box size="0.725 0.600 0.315"/>
             </geometry>
             <material name="red"/>
@@ -15,5 +15,5 @@
         <collision>
             <geometry>
-                <box size="0.7112 0.7112 0.3175"/>
+                <box size="0.725 0.600 0.315"/>
             </geometry>
         </collision>
@@ -25,4 +25,5 @@
     </link>
     <!-- ************ LiDAR Link and Joint ************ -->i
+<!--
     <link name="laser">
 	<visual>
@@ -44,9 +45,11 @@
     </link>
     <joint name="joint_sensor_" type="fixed">
-           <origin xyz="-0.0762 0 0.1905" rpy="0 0 0"/>
+           <origin xyz="0.0025 0 0.1905" rpy="0 0 0"/>
            <parent link="base_link"/>
            <child link="laser"/>
     </joint>
+-->
     <!-- ************ Odometry Link and Joint ************ -->
+<!-- we don't actually need this, it is being broadcasted by encoders.py (odometry tf)
         <link name="odom">
 	<visual>
@@ -68,14 +71,15 @@
     </link>
     <joint name="joint_odom" type="fixed">
-           <origin xyz="0.2 0.2 0.1905" rpy="0 0 0"/>
-           <parent link="base_link"/>
-           <child link="odom"/>
+           <origin xyz="0 0 0" rpy="0 0 0"/>
+           <parent link="odom"/>
+           <child link="base_link"/>
     </joint>
+    -->
     <!-- ************ Wheels and Caster Wheels ************ -->
     <xacro:caster name="right_caster"/>
-    <xacro:caster_joint name="right_caster_joint" parent="base_link" child="right_caster" origin_xyz="0.4 0.3675 0"/>
+    <xacro:caster_joint name="right_caster_joint" parent="base_link" child="right_caster" origin_xyz="0.3625 0.3 0"/>
     <!--<xacro:trasmission_macro name="right_caster_transmission" joint="right_caster_joint" actuator="left_wheel_actuator1"/> -->
     <xacro:caster name="left_caster"/>
-    <xacro:caster_joint name="left_caster_joint" parent="base_link" child="left_caster" origin_xyz="0.4 -0.3675 0"/>
+    <xacro:caster_joint name="left_caster_joint" parent="base_link" child="left_caster" origin_xyz="0.3625 -0.3 0"/>
     <!--<xacro:trasmission_macro name="left_caster_transmission" joint="left_caster_joint" actuator="left_wheel_actuator2"/> -->
     <xacro:link_wheel name="back_left_wheel"/>

Commit message: updated urdf

File: mpdr/urdf/mpdr.xacro (robot description, xacro)
@@ -2,7 +2,7 @@
 <robot name="mpdr" xmlns:xacro="http://www.ros.org/wiki/xacro">
 	<!-- CHANGE TO YOUR PACKAGE NAME -->
-	<xacro:include filename="$(find qusai_test)/urdf/macros.xacro" />
-	<xacro:include filename="$(find qusai_test)/urdf/materials.xacro" />
-	<xacro:include filename="$(find qusai_test)/urdf/mpdr.gazebo" />
+	<xacro:include filename="$(find mpdr)/urdf/macros.xacro" />
+	<xacro:include filename="$(find mpdr)/urdf/materials.xacro" />
+	<xacro:include filename="$(find mpdr)/urdf/mpdr.gazebo" />
   <!-- ************ BASE LINK ************ -->
     <link name="base_link">
@@ -12,4 +12,5 @@
             </geometry>
             <material name="red"/>
+            <origin xyz="-0.36 0 0" rpy="0 0 0"/>
         </visual>
         <collision>
@@ -24,4 +25,13 @@
         </inertial>
     </link>
+    <!--
+    <link name="nav_link">
+    </link>
+    <joint name="nav_joint" type="fixed">
+           <origin xyz="-0.25 0 0" rpy="0 0 3.14"/>
+           <parent link="base_link"/>
+           <child link="nav_link"/>
+    </joint>
+    -->
     <!-- ************ LiDAR Link and Joint ************ -->i
 <!--
@@ -78,8 +88,8 @@
     <!-- ************ Wheels and Caster Wheels ************ -->
     <xacro:caster name="right_caster"/>
-    <xacro:caster_joint name="right_caster_joint" parent="base_link" child="right_caster" origin_xyz="0.3625 0.3 0"/>
+    <xacro:caster_joint name="right_caster_joint" parent="base_link" child="right_caster" origin_xyz="-0.725 0.3 0"/>
     <!--<xacro:trasmission_macro name="right_caster_transmission" joint="right_caster_joint" actuator="left_wheel_actuator1"/> -->
     <xacro:caster name="left_caster"/>
-    <xacro:caster_joint name="left_caster_joint" parent="base_link" child="left_caster" origin_xyz="0.3625 -0.3 0"/>
+    <xacro:caster_joint name="left_caster_joint" parent="base_link" child="left_caster" origin_xyz="-0.725 -0.3 0"/>
     <!--<xacro:trasmission_macro name="left_caster_transmission" joint="left_caster_joint" actuator="left_wheel_actuator2"/> -->
     <xacro:link_wheel name="back_left_wheel"/>
@@ -90,8 +100,8 @@
     <!-- <xacro:trasmission_macro name="back_right__wheel_transmission" joint="back_right_wheel_joint" actuator="left_wheel_actuator4"/> -->
     <xacro:link_wheel name="front_left_wheel"/>
-    <xacro:wheel_joint name="front_left_wheel_joint" parent="base_link" child="front_left_wheel" origin_xyz="-0.25 0.35 -0.15"/>
+    <xacro:wheel_joint name="front_left_wheel_joint" parent="base_link" child="front_left_wheel" origin_xyz="0.0 0.35 -0.15"/>
    <!--<xacro:trasmission_macro name="front_left_wheel_transmission" joint="front_left_wheel_joint" actuator="left_wheel_actuator"/> -->
     <xacro:link_wheel name="front_right_wheel"/>
-    <xacro:wheel_joint name="front_right_wheel_joint" parent="base_link" child="front_right_wheel" origin_xyz="-0.25 -0.35 -0.15"/>
+    <xacro:wheel_joint name="front_right_wheel_joint" parent="base_link" child="front_right_wheel" origin_xyz="0.0 -0.35 -0.15"/>
    <!-- <xacro:trasmission_macro name="front_right_wheel_transmission" joint="front_right_wheel_joint" actuator="right_wheel_actuator"/> -->
 </robot>
